File: LightsAndSuch.kicad_sch (KiCad schematic)
At the start: 70 parts, among them J1 Conn_ARM_SWD_TagConnect_TC2030, Q1 AO3400A, Q2 AO3400A, Q3 AO3400A, Q4 AO3400A, U1 STM32F205RBTx, U2 MAX98357A, U3 TPS54202DDC, U4 TPS7A20xxxDQN, U5 CD4081BM, U6 LM555xM, U7 LM555xM, U8 LM555xM

Commit message: footprints selected and grouped
Parts:
- removed C28: 0.1u, symbol Device:C
- removed C29: 100u, symbol Device:C
- removed D4: LED, symbol Device:LED
- removed Q4: AO3400A, Package_TO_SOT_SMD:SOT-23, symbol Transistor_FET:AO3400A
- removed R12, R14: 10k, symbol Device:R
- removed R13: 3.6k, symbol Device:R
- removed U8: LM555xM, Package_SO:SOIC-8_3.9x4.9mm_P1.27mm, symbol Timer:LM555xM
- C1: footprint (none) -> Capacitor_SMD:C_0402_1005Metric
- C10, C11, C12, C13, C14, C15, C16, C17, C18, C19, C2, C20, C21, C22, C23, C24, C25, C26, C27, C3, C4, C5, C6, C7, C8, C9: footprint (none) -> Capacitor_SMD:C_0201_0603Metric
- Cboot1: renamed from 0.1u; value Cboot -> 0.1u; footprint (none) -> Capacitor_SMD:C_0201_0603Metric
- D1, D3, LS1, LS2, LS3: footprint (none) -> Connector_Molex:Molex_Micro-Fit_3.0_43045-0200_2x01_P3.00mm_Horizontal
- L1: footprint (none) -> Inductor_SMD:L_0603_1608Metric
- R1, R10, R11, R15, R18, R19, R2, R20, R21, R22, R3, R4, R5, R6, R7, R8, R9: footprint (none) -> Resistor_SMD:R_0603_1608Metric
- U5: footprint D14 -> Package_DIP:DIP-14_W7.62mm
Connections:
- net HV renamed TSA
Other:
- moved on the sheet: C26, C27, D1, D3, Q2, Q3, R10, R11, R15, R9, U7
