File: LightsAndSuch.kicad_pcb (KiCad board)
At the start: 4 copper layers, 67.3 x 66.4 mm, 79 parts, among them J1 Conn_01x02_Pin, J2 Conn_02x06_Odd_Even, J8 Conn_02x06_Odd_Even, P1 USB_C_Plug_USB2.0, Q1 AO3400A, Q2 AO3400A, Q3 AO3400A, Q4 AO3400A, Q5 AO3400A, U1 RP2040, U2 MAX98357A, U3 TPS54202DDC, U4 LM3940IMP-3.3, U5 CD4081BM, U6 LM555xM, U7 LM555xM, U8 W25Q128JVS, U9 NCP1117-3.3_SOT223

Commit message: need to route test points
Parts:
- removed C9: 1u, Capacitor_SMD:C_0201_0603Metric
- added 1u1: 1u, Capacitor_SMD:C_0603_1608Metric_Pad1.08x0.95mm_HandSolder, F.Cu at (111.4, 80.9)
- added TP1: TestPoint_Probe, S2761-46R:HARWIN_S2761-46R, F.Cu at (89.9, 113.0)
- added TP10: TestPoint_Probe, S2761-46R:HARWIN_S2761-46R, F.Cu at (148.6, 123.3)
- added TP11: TestPoint_Probe, S2761-46R:HARWIN_S2761-46R, F.Cu at (148.6, 125.8)
- added TP2: TestPoint_Probe, S2761-46R:HARWIN_S2761-46R, F.Cu at (107.1, 93.3)
- added TP3: TestPoint_Probe, S2761-46R:HARWIN_S2761-46R, F.Cu at (104.2, 92.8)
- added TP4: TestPoint_Probe, S2761-46R:HARWIN_S2761-46R, F.Cu at (107.7, 103.9)
- added TP5: TestPoint_Probe, S2761-46R:HARWIN_S2761-46R, F.Cu at (145.2, 120.8)
- added TP6: TestPoint_Probe, S2761-46R:HARWIN_S2761-46R, F.Cu at (145.2, 123.3)
- added TP7: TestPoint_Probe, S2761-46R:HARWIN_S2761-46R, F.Cu at (145.2, 125.8)
- added TP8: TestPoint_Probe, S2761-46R:HARWIN_S2761-46R, F.Cu at (144.8, 117.3)
- added TP9: TestPoint_Probe, S2761-46R:HARWIN_S2761-46R, F.Cu at (148.6, 120.8)
- C1: footprint Capacitor_SMD:C_0402_1005Metric -> Capacitor_SMD:C_0603_1608Metric_Pad1.08x0.95mm_HandSolder
- C10, C11, C12, C13, C14, C15, C16, C17, C18, C19, C2, C20, C21, C22, C23, C24, C25, C26, C27, C3, C31, C32, C33, C4, C5, C6, Cboot1: footprint Capacitor_SMD:C_0201_0603Metric -> Capacitor_SMD:C_0603_1608Metric_Pad1.08x0.95mm_HandSolder
- C28: value C -> 1u; footprint Capacitor_SMD:C_0201_0603Metric -> Capacitor_SMD:C_0603_1608Metric_Pad1.08x0.95mm_HandSolder
- C29, C30: value C -> 100n; footprint Capacitor_SMD:C_0201_0603Metric -> Capacitor_SMD:C_0603_1608Metric_Pad1.08x0.95mm_HandSolder
- C7, C8: footprint Capacitor_SMD:C_0603_1608Metric -> Capacitor_SMD:C_0603_1608Metric_Pad1.08x0.95mm_HandSolder
- R1, R10, R11, R12, R13, R14, R15, R16, R17, R18, R19, R2, R20, R21, R22, R3, R4, R5, R6, R7, R8, R9: footprint Resistor_SMD:R_0603_1608Metric -> Resistor_SMD:R_0603_1608Metric_Pad0.98x0.95mm_HandSolder
- moved C11 137.0 mm to (1.68, 0.76)
- moved C28 13.8 mm to (111.2, 93.7), turned to -90 degrees
- moved C30 5.93 mm to (114.8, 79.3), turned to 0 degrees
- moved C29 5.64 mm to (114.8, 77.8), turned to 0 degrees
- moved C3 5.46 mm to (81.5, 93.1), turned to -90 degrees
- moved C10 4.60 mm to (114.8, 84.0), turned to 0 degrees
- moved C18 4.28 mm to (99.8, 94.7), turned to -90 degrees
- moved C13 3.93 mm to (114.8, 80.9), turned to 0 degrees
- moved C5 3.92 mm to (83.1, 93.2), turned to -90 degrees
- moved C17 3.57 mm to (101.5, 94.7), turned to -90 degrees
- moved C24 2.64 mm to (115.0, 120.2)
- moved C14 2.47 mm to (109.6, 93.7), turned to -90 degrees
- moved R6 2.41 mm to (87.9, 112.2), turned to 90 degrees
- moved C12 2.22 mm to (114.8, 82.4)
- moved C16 1.94 mm to (114.1, 85.6), turned to 0 degrees
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Routing:
- net GND: track 61.8 -> 43.8 mm, vias 58 -> 63
- net Trigger: track 74.4 -> 60.2 mm
- net Net-(U1-VREG_VOUT): track 17.8 -> 31.0 mm
- net +3.3V: track 78.2 -> 81.8 mm, vias 9 -> 7
- net /USB_D+: track 21.0 -> 24.3 mm
- net +5V: track 116.6 -> 119.2 mm, vias 6 -> 3
- net Net-(U1-GPIO10): track 7.57 -> 6.20 mm
- net Net-(U3-BOOT): track 4.49 -> 3.48 mm
- net Net-(U3-FB): track 8.60 -> 7.62 mm
- net Net-(U7-TR): track 5.51 -> 4.53 mm
- net Net-(Q5-G): track 5.00 -> 4.12 mm
- net TSA: track 21.2 -> 22.0 mm
- net +12V: track 98.0 -> 97.3 mm
- net IMD_Fault: track 10.7 -> 11.4 mm
- net Break: track 28.8 -> 29.4 mm
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