File: LightsAndSuch.kicad_pcb (KiCad board)
At the start: 4 copper layers, 67.3 x 66.4 mm, 87 parts, among them J1 Conn_01x02_Pin, J2 Conn_02x06_Odd_Even, J8 Conn_02x06_Odd_Even, P1 USB_C_Plug_USB2.0, Q1 AO3400A, Q2 AO3400A, Q3 AO3400A, Q4 AO3400A, Q5 AO3400A, U1 RP2040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

Commit message: changes from aiden's computer
Parts:
- moved R26 27.4 mm to (102.0, 90.2), turned to 180 degrees
Routing:
- net +3.3V: track 70.2 -> 73.1 mm, vias 6 -> 4
- net /nSD_MODE: track 7.23 -> 8.87 mm, vias 0 -> 2
- net Net-(U1-XIN): track 24.0 -> 25.6 mm
